File: USB_TO_UART.kicad_sch (KiCad schematic)
At the start: 9 parts, among them U3 FT232RL

Commit message: PCB preview on KiCanvas wasnt working
Parts:
- D5: value LED -> TXLED
- D6: value LED -> RXLED
Changed lines of the file:
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@@
 			)
 		)
-		(property "Value" "LED"
+		(property "Value" "TXLED"
 			(at 154.6225 110.49 0)
 			(show_name no)
@@
 			)
 		)
-		(property "Value" "LED"
+		(property "Value" "RXLED"
 			(at 163.5125 113.03 0)
 			(show_name no)
